File: Pentax-S5z-LED-ring.sch (KiCad schematic (older format))
At the start: 46 parts, among them IC1 ATTINY13-S, P1 CONN_2, P2 +, P3 -, P4 CONN_2, Q1 MOSFET_N, SW1 SW_PUSH, SW2 SW_PUSH

Commit message: 68R it is.
Parts:
- R1, R10, R11, R12, R13, R14, R15, R16, R2, R3, R4, R5, R6, R7, R8, R9: value 65R -> 68R
Other:
- note added: "WW: 3.29V @ 26mA - 25mA --> 68R (5V)\n W: 3.19V @ 28mA - 25mA --> 68R (5V)"
- note removed: "WW: 3.29V --> 26mA --> 65R (5V)\n W: 3.19V --> 28mA --> 65R (5V)"
Changed lines of the file:
@@
-EESchema Schematic File Version 2  date Mon 29 Apr 2013 01:08:56 AM CEST
+EESchema Schematic File Version 2  date Mon 29 Apr 2013 02:40:01 AM CEST
 LIBS:my_parts
 LIBS:power
@@
 Sheet 1 1
 Title "Pentax S5z LED ring"
-Date "28 apr 2013"
+Date "29 apr 2013"
 Rev "1.0"
 Comp "2013 - blog.spitzenpfeil.org"
@@
 P 6300 1850
 F 0 "R1" V 6380 1850 50  0000 C CNN
-F 1 "65R" V 6300 1850 50  0000 C CNN
+F 1 "68R" V 6300 1850 50  0000 C CNN
 F 2 "" H 6300 1850 60  0000 C CNN
 F 3 "" H 6300 1850 60  0000 C CNN
@@
 P 6600 1850
 F 0 "R2" V 6680 1850 50  0000 C CNN
-F 1 "65R" V 6600 1850 50  0000 C CNN
+F 1 "68R" V 6600 1850 50  0000 C CNN
 F 2 "" H 6600 1850 60  0000 C CNN
 F 3 "" H 6600 1850 60  0000 C CNN
@@
 P 6900 1850
 F 0 "R3" V 6980 1850 50  0000 C CNN
-F 1 "65R" V 6900 1850 50  0000 C CNN
+F 1 "68R" V 6900 1850 50  0000 C CNN
 F 2 "" H 6900 1850 60  0000 C CNN
 F 3 "" H 6900 1850 60  0000 C CNN
@@
 P 7200 1850
 F 0 "R4" V 7280 1850 50  0000 C CNN
-F 1 "65R" V 7200 1850 50  0000 C CNN
+F 1 "68R" V 7200 1850 50  0000 C CNN
 F 2 "" H 7200 1850 60  0000 C CNN
 F 3 "" H 7200 1850 60  0000 C CNN
@@
 P 7500 1850
 F 0 "R5" V 7580 1850 50  0000 C CNN
-F 1 "65R" V 7500 1850 50  0000 C CNN
+F 1 "68R" V 7500 1850 50  0000 C CNN
 F 2 "" H 7500 1850 60  0000 C CNN
 F 3 "" H 7500 1850 60  0000 C CNN
@@
 P 7800 1850
 F 0 "R6" V 7880 1850 50  0000 C CNN
-F 1 "65R" V 7800 1850 50  0000 C CNN
+F 1 "68R" V 7800 1850 50  0000 C CNN
 F 2 "" H 7800 1850 60  0000 C CNN
 F 3 "" H 7800 1850 60  0000 C CNN
@@
 P 8100 1850
 F 0 "R7" V 8180 1850 50  0000 C CNN
-F 1 "65R" V 8100 1850 50  0000 C CNN
+F 1 "68R" V 8100 1850 50  0000 C CNN
 F 2 "" H 8100 1850 60  0000 C CNN
 F 3 "" H 8100 1850 60  0000 C CNN
@@
 P 8400 1850
 F 0 "R8" V 8480 1850 50  0000 C CNN
-F 1 "65R" V 8400 1850 50  0000 C CNN
+F 1 "68R" V 8400 1850 50  0000 C CNN
 F 2 "" H 8400 1850 60  0000 C CNN
 F 3 "" H 8400 1850 60  0000 C CNN
@@
 P 8700 1850
 F 0 "R9" V 8780 1850 50  0000 C CNN
-F 1 "65R" V 8700 1850 50  0000 C CNN
+F 1 "68R" V 8700 1850 50  0000 C CNN
 F 2 "" H 8700 1850 60  0000 C CNN
 F 3 "" H 8700 1850 60  0000 C CNN
@@
 P 9000 1850
 F 0 "R10" V 9080 1850 50  0000 C CNN
-F 1 "65R" V 9000 1850 50  0000 C CNN
+F 1 "68R" V 9000 1850 50  0000 C CNN
 F 2 "" H 9000 1850 60  0000 C CNN
 F 3 "" H 9000 1850 60  0000 C CNN
@@
 P 9300 1850
 F 0 "R11" V 9380 1850 50  0000 C CNN
-F 1 "65R" V 9300 1850 50  0000 C CNN
+F 1 "68R" V 9300 1850 50  0000 C CNN
 F 2 "" H 9300 1850 60  0000 C CNN
 F 3 "" H 9300 1850 60  0000 C CNN
@@
 P 9600 1850
 F 0 "R12" V 9680 1850 50  0000 C CNN
-F 1 "65R" V 9600 1850 50  0000 C CNN
+F 1 "68R" V 9600 1850 50  0000 C CNN
 F 2 "" H 9600 1850 60  0000 C CNN
 F 3 "" H 9600 1850 60  0000 C CNN
@@
 P 9900 1850
 F 0 "R13" V 9980 1850 50  0000 C CNN
-F 1 "65R" V 9900 1850 50  0000 C CNN
+F 1 "68R" V 9900 1850 50  0000 C CNN
 F 2 "" H 9900 1850 60  0000 C CNN
 F 3 "" H 9900 1850 60  0000 C CNN
@@
 P 10200 1850
 F 0 "R14" V 10280 1850 50  0000 C CNN
-F 1 "65R" V 10200 1850 50  0000 C CNN
+F 1 "68R" V 10200 1850 50  0000 C CNN
 F 2 "" H 10200 1850 60  0000 C CNN
 F 3 "" H 10200 1850 60  0000 C CNN
@@
 P 10500 1850
 F 0 "R15" V 10580 1850 50  0000 C CNN
-F 1 "65R" V 10500 1850 50  0000 C CNN
+F 1 "68R" V 10500 1850 50  0000 C CNN
 F 2 "" H 10500 1850 60  0000 C CNN
 F 3 "" H 10500 1850 60  0000 C CNN
@@
 P 10800 1850
 F 0 "R16" V 10880 1850 50  0000 C CNN
-F 1 "65R" V 10800 1850 50  0000 C CNN
+F 1 "68R" V 10800 1850 50  0000 C CNN
 F 2 "" H 10800 1850 60  0000 C CNN
 F 3 "" H 10800 1850 60  0000 C CNN
@@
 	1500 4650 1500 4800
 Connection ~ 1500 4650
-Text Notes 4250 1550 0    60   ~ 0
-WW: 3.29V --> 26mA --> 65R (5V)\n  W: 3.19V --> 28mA -->  65R (5V)
+Text Notes 4000 1550 0    60   ~ 0
+WW: 3.29V @ 26mA  - 25mA --> 68R (5V)\n  W: 3.19V @ 28mA - 25mA  -->  68R (5V)
 $EndSCHEMATC
