File: Pentax-S5z-LED-ring.sch (KiCad schematic (older format))
At the start: 46 parts, among them IC1 ATTINY13-S, P1 CONN_2, P2 +, P3 -, P4 CONN_2, Q1 MOSFET_N, SW1 SW_PUSH, SW2 SW_PUSH

Commit message: Switched ATtiny13 to DFN10 package.
Had to move to KiCAD's new way of handling footprint libraries.
Parts:
- removed IC1: ATTINY13-S, SO8-200, symbol ATTINY13-S
- added IC1: MADW__ATTINY13-MM, MADW__MLF10, symbol MADW__ATTINY13-MM
Connections:
- net +5V: now also IC1.10 (VCC)
- net GND: now also IC1.5 (GND), IC1.PAD (GND)
- net MISO: now also IC1.7 (PB1(MISO/AIN1/OC0B/INT0/PCINT1))
- net PWM: now also IC1.6 (PB0(MOSI/AIN0/OC0A/PCINT0))
- net RESET: now also IC1.1 (PB5(~RESET~/ADC0/PCINT5/dW))
- net SCK: now also IC1.9 (PB2(SCK/ADC1/T0/PCINT2))
Changed lines of the file:
@@
-EESchema Schematic File Version 2  date Mon 29 Apr 2013 02:40:01 AM CEST
+EESchema Schematic File Version 2
 LIBS:my_parts
 LIBS:power
@@
 Sheet 1 1
 Title "Pentax S5z LED ring"
-Date "29 apr 2013"
-Rev "1.0"
+Date "13 Dec 2013"
+Rev "1.01"
 Comp "2013 - blog.spitzenpfeil.org"
 Comment1 ""
@@
 	9000 2100 9000 2200
 Connection ~ 9000 2200
-$Comp
-L ATTINY13-S IC1
-U 1 1 51640F05
-P 3150 3550
-F 0 "IC1" H 3250 3600 60  0000 C CNN
-F 1 "ATTINY13-S" H 4450 2800 60  0000 C CNN
-F 2 "SO8-200" H 3400 2800 60  0001 C CNN
-F 3 "" H 3150 3550 60  0000 C CNN
-	1    3150 3550
-	1    0    0    -1
-$EndComp
 $Comp
 L R R17
@@
 Text Notes 4000 1550 0    60   ~ 0
 WW: 3.29V @ 26mA  - 25mA --> 68R (5V)\n  W: 3.19V @ 28mA - 25mA  -->  68R (5V)
+$Comp
+L MADW__ATTINY13-MM IC1
+U 1 1 52AB21C7
+P 3950 3900
+F 0 "IC1" H 3250 4300 60  0000 C CNN
+F 1 "MADW__ATTINY13-MM" H 4300 3500 60  0000 C CNN
+F 2 "MADW__MLF10" H 3450 3500 60  0000 C CNN
+F 3 "" H 3150 4250 60  0000 C CNN
+	1    3950 3900
+	1    0    0    -1
+$EndComp
+Wire Wire Line
+	4950 4050 4950 4150
 $EndSCHEMATC
